Commit message: feat: update dimensions for bin base and wheels in URDF files

File: bin_description/urdf/body/bin_base.urdf.xacro (robot description, xacro)
@@ -1,6 +1,6 @@
 <?xml version="1.0"?>
 <robot xmlns:xacro="http://www.ros.org/wiki/xacro">
-<xacro:property name="base_width" value="0.227" />
-<xacro:property name="base_length" value="0.224725" />
+<xacro:property name="base_width" value="0.2055" />
+<xacro:property name="base_length" value="0.2052" />
 <xacro:property name="base_height" value="0.12" />
 <!-- <xacro:property name="base_height" value="0.140234" /> -->

File: bin_description/urdf/body/bin_wheels.urdf.xacro (robot description, xacro)
@@ -2,6 +2,6 @@
 <robot xmlns:xacro="http://www.ros.org/wiki/xacro">
     <xacro:property name="rubber_density" value="1100.0" />
-    <xacro:property name="wheel_width" value="0.0214" />
-    <xacro:property name="wheel_radius" value="0.031755" />
+    <xacro:property name="wheel_width" value="0.0260" />
+    <xacro:property name="wheel_radius" value="0.0335" />
     <xacro:property name="wheel_mass" value="${rubber_density * pi * wheel_radius * wheel_radius * wheel_width}" />
     <xacro:property name="motor_mass"  value="0.333" />
