Commit message: Smart waste bin update

File: bin_description/urdf/body/bin_cover.urdf.xacro (robot description, xacro)
@@ -33,10 +33,10 @@
             </inertial>
         </link>
-        <joint name="${prefix}bin_cover_joint" type="revolute">
+        <joint name="${prefix}bin_cover_joint" type="fixed">
             <parent link="${prefix}bin_top_link"/>
             <child link="${prefix}bin_cover_link"/>
             <origin xyz="${-cover_length/2} 0 ${bin_height}" rpy="0 0 0"/>
-            <axis xyz="0 1 0"/>
-            <limit lower="${-pi/2}" upper="0" effort="100" velocity="1.0"/>
+            <!-- <axis xyz="0 1 0"/>
+            <limit lower="${-pi/2}" upper="0" effort="100" velocity="1.0"/> -->
         </joint>
     </xacro:macro>

File: bin_description/urdf/ros2_control/bin_ros2_control.xacro (robot description, xacro)
@@ -54,5 +54,5 @@
                 <state_interface name="linear_acceleration.z"/>
             </sensor> -->
-            <joint name="${prefix}bin_cover_joint">
+            <!-- <joint name="${prefix}bin_cover_joint">
                 <command_interface name="position">
                     <param name="min">${-pi/2}</param>
@@ -61,5 +61,5 @@
                 <state_interface name="position"/>
                 <state_interface name="velocity"/>
-            </joint>
+            </joint> -->
         </ros2_control>
     </xacro:macro>
